Commit message: developed navigation parts.   - nav to object   - approach object   - nav to room   - find target   - nav to target   - approach target   - go back to start point

File: tb3_mobile_manipulation_description/urdf/tb3_mobile_manipulation.base.gazebo.xacro (robot description, xacro)
@@ -8,6 +8,6 @@
   </gazebo>
   <gazebo reference="wheel_left_link">
-    <mu1>0.1</mu1>
-    <mu2>0.1</mu2>
+    <mu1>10000</mu1>
+    <mu2>10000</mu2>
     <kp>500000.0</kp>
     <kd>10.0</kd>
@@ -18,6 +18,6 @@
   </gazebo>
   <gazebo reference="wheel_right_link">
-    <mu1>0.1</mu1>
-    <mu2>0.1</mu2>
+    <mu1>10000</mu1>
+    <mu2>10000</mu2>
     <kp>500000.0</kp>
     <kd>10.0</kd>

File: tb3_mobile_manipulation_description/urdf/tb3_mobile_manipulation.base.urdf.xacro (robot description, xacro)
@@ -28,7 +28,10 @@
         <mass value="2.7771056e+00"/>
         <!-- <mass value="1.7771056e+00"/> -->
-        <inertia ixx="1.8257500e-01" ixy="4.9296089e-03" ixz="-1.1606178e-05"
-                 iyy="4.8786869e-02" iyz="1.4954898e-05"
-                 izz="3.9852748e-02" />
+        <!-- <inertia ixx="1.8257500e-01" ixy="4.9296089e-03" ixz="-1.1606178e-05" -->
+                 <!-- iyy="4.8786869e-02" iyz="1.4954898e-05" -->
+                 <!-- izz="3.9852748e-02" /> -->
+        <inertia ixx="1" ixy="0" ixz="0"
+                 iyy="1" iyz="0"
+                 izz="1" />
       </inertial>
     </link>

File: tb3_mobile_manipulation_description/urdf/tb3_mobile_manipulation.manipulator.gazebo.xacro (robot description, xacro)
@@ -28,6 +28,14 @@
   <!-- gripper_link -->
   <RefLink ref="gripper_link"/>
+  <gazebo reference="gripper_link">
+    <turnGravityOff>true</turnGravityOff>
+    <implicitSpringDamper>1</implicitSpringDamper>
+  </gazebo>
   <!-- gripper_link_sub -->
   <RefLink ref="gripper_link_sub"/>
+  <gazebo reference="gripper_link_sub">
+    <turnGravityOff>true</turnGravityOff>
+    <implicitSpringDamper>1</implicitSpringDamper>
+  </gazebo>
   <!-- end effector link -->
   <gazebo reference="end_effector_link">
